File: EEOP_Display/EEOP_Display.kicad_sch (KiCad schematic)
At the start: 2 parts, among them J1 Conn_01x32, J2 Conn_01x32

Commit message: Finished EEOP PCB
Parts:
- removed J1: Conn_01x32, Connector_FFC-FPC:Hirose_FH12-32S-0.5SH_1x32-1MP_P0.50mm_Horizontal, symbol Connector_Generic:Conn_01x32
- added J1: FH34SRJ-32S-0.5SH_50_, Touchpoint:HRS_FH34SRJ-32S-0.5SH_50_, symbol FH34SRJ-32S-0.5SH_50_:FH34SRJ-32S-0.5SH_50_
Connections:
- net E1: now also J1.1
- net E10: now also J1.10
- net E11: now also J1.11
- net E12: now also J1.12
- net E13: now also J1.13
- net E14: now also J1.14
- net E15: now also J1.15
- net E16: now also J1.16
- net E17: now also J1.17
- net E18: now also J1.18
- net E19: now also J1.19
- net E2: now also J1.2
- net E20: now also J1.20
- net E21: now also J1.21
- net E22: now also J1.22
- net E23: now also J1.23
- net E24: now also J1.24
- net E25: now also J1.25
- net E26: now also J1.26
- net E27: now also J1.27
- net E28: now also J1.28
- net E29: now also J1.29
- net E3: now also J1.3
- net E30: now also J1.30
- net E31: now also J1.31
- net E32: now also J1.32
- net E4: now also J1.4
- net E5: now also J1.5
- net E6: now also J1.6
- net E7: now also J1.7
- net E8: now also J1.8
- net E9: now also J1.9
- new net: J1.S1 (SHIELD), J1.S2 (SHIELD)
- no-connect marks 0 -> 1
Changed lines of the file:
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@@
 	(generator_version "9.0")
 	(paper "A4")
+	(no_connect
+		(at 128.27 118.11)
+	)
 	(label "E17"
 		(at 107.95 74.93 0)
@@
 	)
 	(symbol
-		(lib_id "Connector_Generic:Conn_01x32")
-		(at 102.87 74.93 180)
+		(lib_id "FH34SRJ-32S-0.5SH_50_:FH34SRJ-32S-0.5SH_50_")
+		(at 118.11 74.93 0)
 		(unit 1)
 		(exclude_from_sim no)
@@
 		(fields_autoplaced yes)
 		(property "Reference" "J1"
-			(at 102.87 27.94 0)
-			(effects
-				(font
-					(size 1.27 1.27)
-				)
-			)
-		)
-		(property "Value" "Conn_01x32"
-			(at 102.87 30.48 0)
-			(effects
-				(font
-					(size 1.27 1.27)
-				)
-			)
-		)
-		(property "Footprint" "Connector_FFC-FPC:Hirose_FH12-32S-0.5SH_1x32-1MP_P0.50mm_Horizontal"
-			(at 102.87 74.93 0)
-			(effects
-				(font
-					(size 1.27 1.27)
-				)
-				(hide yes)
-			)
-		)
-		(property "Datasheet" "~"
-			(at 102.87 74.93 0)
-			(effects
-				(font
-					(size 1.27 1.27)
-				)
-				(hide yes)
-			)
-		)
-		(property "Description" "Generic connector, single row, 01x32, script generated (kicad-library-utils/schlib/autogen/connector/)"
-			(at 102.87 74.93 0)
-			(effects
-				(font
-					(size 1.27 1.27)
-				)
-				(hide yes)
-			)
+			(at 118.11 26.67 0)
+			(effects
+				(font
+					(size 1.27 1.27)
+				)
+			)
+		)
+		(property "Value" "FH34SRJ-32S-0.5SH_50_"
+			(at 118.11 29.21 0)
+			(effects
+				(font
+					(size 1.27 1.27)
+				)
+			)
+		)
+		(property "Footprint" "Touchpoint:HRS_FH34SRJ-32S-0.5SH_50_"
+			(at 118.11 74.93 0)
+			(effects
+				(font
+					(size 1.27 1.27)
+				)
+				(justify bottom)
+				(hide yes)
+			)
+		)
+		(property "Datasheet" ""
+			(at 118.11 74.93 0)
+			(effects
+				(font
+					(size 1.27 1.27)
+				)
+				(hide yes)
+			)
+		)
+		(property "Description" ""
+			(at 118.11 74.93 0)
+			(effects
+				(font
+					(size 1.27 1.27)
+				)
+				(hide yes)
+			)
+		)
+		(property "DigiKey_Part_Number" "26-FH34SRJ-32S-0.5SH(50)CT-ND"
+			(at 118.11 74.93 0)
+			(effects
+				(font
+					(size 1.27 1.27)
+				)
+				(justify bottom)
+				(hide yes)
+			)
+		)
+		(property "SnapEDA_Link" "https://www.snapeda.com/parts/FH34SRJ-32S-0.5SH(50)/Hirose+Electric+Co+Ltd/view-part/?ref=snap"
+			(at 118.11 74.93 0)
+			(effects
+				(font
+					(size 1.27 1.27)
+				)
+				(justify bottom)
+				(hide yes)
+			)
+		)
+		(property "Description_1" "32 Position FFC, FPC Connector Contacts, Top and Bottom 0.020 (0.50mm) Surface Mount, Right Angle"
+			(at 118.11 74.93 0)
+			(effects
+				(font
+					(size 1.27 1.27)
+				)
+				(justify bottom)
+				(hide yes)
+			)
+		)
+		(property "Package" "None"
+			(at 118.11 74.93 0)
+			(effects
+				(font
+					(size 1.27 1.27)
+				)
+				(justify bottom)
+				(hide yes)
+			)
+		)
+		(property "Check_prices" "https://www.snapeda.com/parts/FH34SRJ-32S-0.5SH(50)/Hirose+Electric+Co+Ltd/view-part/?ref=eda"
+			(at 118.11 74.93 0)
+			(effects
+				(font
+					(size 1.27 1.27)
+				)
+				(justify bottom)
+				(hide yes)
+			)
+		)
+		(property "MF" "Hirose Electric Co Ltd"
+			(at 118.11 74.93 0)
+			(effects
+				(font
+					(size 1.27 1.27)
+				)
+				(justify bottom)
+				(hide yes)
+			)
+		)
+		(property "MP" "FH34SRJ-32S-0.5SH(50)"
+			(at 118.11 74.93 0)
+			(effects
+				(font
+					(size 1.27 1.27)
+				)
+				(justify bottom)
+				(hide yes)
+			)
+		)
+		(property "MANUFACTURER" "HRS"
+			(at 118.11 74.93 0)
+			(effects
+				(font
+					(size 1.27 1.27)
+				)
+				(justify bottom)
+				(hide yes)
+			)
+		)
+		(pin "5"
+		)
+		(pin "6"
+		)
+		(pin "1"
+		)
+		(pin "8"
+		)
+		(pin "10"
+		)
+		(pin "2"
+		)
+		(pin "3"
+		)
+		(pin "4"
+		)
+		(pin "7"
+		)
+		(pin "9"
+		)
+		(pin "14"
+		)
+		(pin "29"
+		)
+		(pin "18"
+		)
+		(pin "S1"
+		)
+		(pin "12"
+		)
+		(pin "28"
+		)
+		(pin "31"
+		)
+		(pin "17"
+		)
+		(pin "20"
 		)
 		(pin "11"
 		)
-		(pin "12"
-		)
-		(pin "1"
-		)
-		(pin "4"
-		)
-		(pin "6"
-		)
-		(pin "7"
-		)
-		(pin "3"
-		)
-		(pin "8"
-		)
-		(pin "9"
-		)
-		(pin "10"
-		)
-		(pin "18"
+		(pin "15"
+		)
+		(pin "21"
+		)
+		(pin "23"
+		)
+		(pin "27"
+		)
+		(pin "19"
+		)
+		(pin "13"
+		)
+		(pin "22"
+		)
+		(pin "16"
+		)
+		(pin "25"
+		)
+		(pin "26"
+		)
+		(pin "24"
 		)
 		(pin "30"
 		)
-		(pin "31"
-		)
-		(pin "21"
-		)
-		(pin "2"
-		)
-		(pin "5"
-		)
-		(pin "19"
-		)
-		(pin "22"
-		)
-		(pin "24"
-		)
-		(pin "14"
-		)
-		(pin "15"
-		)
-		(pin "25"
-		)
-		(pin "27"
-		)
-		(pin "17"
-		)
-		(pin "23"
-		)
-		(pin "13"
-		)
-		(pin "26"
-		)
-		(pin "16"
-		)
-		(pin "28"
-		)
-		(pin "20"
-		)
-		(pin "29"
-		)
 		(pin "32"
 		)
+		(pin "S2"
+		)
 		(instances
