File: Touchpoint_Mainboard/Touchpoint_Mainboard.kicad_sch (KiCad schematic)
At the start: 31 parts, among them J101 Conn_01x02, U101 RP2040, U102 NCP1117-3.3_SOT223, U103 W25Q128JVS, Y101 ABM8-272-T3

Commit message: Final manufacturing adjustments
Parts:
- C103, C105: footprint Capacitor_SMD:C_0402_1005Metric -> Capacitor_SMD:C_0805_2012Metric
Other:
- sheet Buttons ports: added RCLICK, SCROLLA, SCROLLB; removed none
Changed lines of the file:
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@@
 	)
 	(label "~{BOOT}"
-		(at 146.05 113.03 0)
+		(at 146.05 109.22 0)
 		(effects
 			(font
@@
 	)
 	(label "GPIO3"
-		(at 142.24 137.16 0)
+		(at 142.24 138.43 0)
 		(effects
 			(font
@@
 	)
 	(label "~{RESET}"
-		(at 146.05 118.11 0)
+		(at 146.05 114.3 0)
 		(effects
 			(font
@@
 	)
 	(label "GPIO27"
-		(at 149.86 99.06 0)
+		(at 149.86 96.52 0)
 		(effects
 			(font
@@
 	)
 	(label "GPIO4"
-		(at 142.24 142.24 0)
+		(at 142.24 143.51 0)
 		(effects
 			(font
@@
 	)
 	(label "GPIO13"
-		(at 146.05 115.57 0)
+		(at 146.05 111.76 0)
 		(effects
 			(font
@@
 	)
 	(label "GPIO26"
-		(at 149.86 96.52 0)
+		(at 149.86 93.98 0)
+		(effects
+			(font
+				(size 1.27 1.27)
+			)
+			(justify left bottom)
+		)
+	)
+	(label "GPIO17"
+		(at 146.05 119.38 0)
 		(effects
 			(font
@@
 		)
 	)
+	(label "GPIO16"
+		(at 146.05 116.84 0)
+		(effects
+			(font
+				(size 1.27 1.27)
+			)
+			(justify left bottom)
+		)
+	)
 	(label "GPIO5"
-		(at 142.24 129.54 0)
+		(at 142.24 130.81 0)
 		(effects
 			(font
@@
 	)
 	(label "GPIO0"
-		(at 142.24 134.62 0)
+		(at 142.24 135.89 0)
 		(effects
 			(font
@@
 	)
 	(label "GPIO2"
-		(at 142.24 139.7 0)
+		(at 142.24 140.97 0)
 		(effects
 			(font
@@
 	)
 	(label "GPIO1"
-		(at 142.24 132.08 0)
+		(at 142.24 133.35 0)
 		(effects
 			(font
@@
 	)
 	(label "GPIO15"
-		(at 149.86 101.6 0)
+		(at 149.86 99.06 0)
+		(effects
+			(font
+				(size 1.27 1.27)
+			)
+			(justify left bottom)
+		)
+	)
+	(label "GPIO18"
+		(at 146.05 121.92 0)
 		(effects
 			(font
@@
 			)
 		)
-		(property "Footprint" "Capacitor_SMD:C_0402_1005Metric"
+		(property "Footprint" "Capacitor_SMD:C_0805_2012Metric"
 			(at 36.5252 48.26 0)
 			(effects
@@
 			)
 		)
-		(property "Footprint" "Capacitor_SMD:C_0402_1005Metric"
+		(property "Footprint" "Capacitor_SMD:C_0805_2012Metric"
 			(at 91.1352 48.26 0)
 			(effects
@@
 	)
 	(sheet
-		(at 123.19 127)
+		(at 123.19 128.27)
 		(size 19.05 19.05)
 		(exclude_from_sim no)
@@
 		)
 		(property "Sheetname" "PMW3389"
-			(at 123.19 126.2884 0)
+			(at 123.19 127.5584 0)
 			(effects
 				(font
@@
 		)
 		(property "Sheetfile" "PMW3389.kicad_sch"
-			(at 123.19 146.6346 0)
+			(at 123.19 147.9046 0)
 			(effects
 				(font
@@
 		)
 		(pin "CS" input
-			(at 142.24 129.54 0)
+			(at 142.24 130.81 0)
 			(effects
 				(font
@@
 		)
 		(pin "INT" input
-			(at 142.24 132.08 0)
+			(at 142.24 133.35 0)
 			(effects
 				(font
@@
 		)
 		(pin "MISO" input
-			(at 142.24 134.62 0)
+			(at 142.24 135.89 0)
 			(effects
 				(font
@@
 		)
 		(pin "MOSI" input
-			(at 142.24 137.16 0)
+			(at 142.24 138.43 0)
 			(effects
 				(font
@@
 		)
 		(pin "SCLK" input
-			(at 142.24 139.7 0)
+			(at 142.24 140.97 0)
 			(effects
 				(font
@@
 		)
 		(pin "~{RST}" input
-			(at 142.24 142.24 0)
+			(at 142.24 143.51 0)
 			(effects
 				(font
@@
 	)
 	(sheet
-		(at 123.19 110.49)
-		(size 22.86 10.16)
+		(at 123.19 106.68)
+		(size 22.86 16.51)
 		(exclude_from_sim no)
 		(in_bom yes)
@@
 		)
 		(property "Sheetname" "Buttons"
-			(at 123.19 109.7784 0)
+			(at 123.19 105.9684 0)
 			(effects
 				(font
@@
 		)
 		(property "Sheetfile" "Buttons.kicad_sch"
-			(at 123.19 121.2346 0)
+			(at 123.19 123.7746 0)
 			(effects
 				(font
@@
 		)
 		(pin "~{BOOT}" input
-			(at 146.05 113.03 0)
+			(at 146.05 109.22 0)
 			(effects
 				(font
@@
 		)
 		(pin "~{RESET}" input
-			(at 146.05 118.11 0)
+			(at 146.05 114.3 0)
 			(effects
 				(font
@@
 		)
 		(pin "~{LCLICK}" input
-			(at 146.05 115.57 0)
+			(at 146.05 111.76 0)
+			(effects
+				(font
+					(size 1.27 1.27)
+				)
+				(justify right)
+			)
+		)
+		(pin "RCLICK" input
+			(at 146.05 116.84 0)
+			(effects
+				(font
+					(size 1.27 1.27)
+				)
+				(justify right)
+			)
+		)
+		(pin "SCROLLA" input
+			(at 146.05 119.38 0)
+			(effects
+				(font
+					(size 1.27 1.27)
+				)
+				(justify right)
+			)
+		)
+		(pin "SCROLLB" input
+			(at 146.05 121.92 0)
 			(effects
 				(font
@@
 	)
 	(sheet
-		(at 123.19 93.98)
+		(at 123.19 91.44)
 		(size 26.67 10.16)
 		(exclude_from_sim no)
@@
 		)
 		(property "Sheetname" "Zoom_Wheel"
-			(at 123.19 93.2684 0)
+			(at 123.19 90.7284 0)
 			(effects
 				(font
@@
 		)
 		(property "Sheetfile" "Zoom_Wheel.kicad_sch"
-			(at 123.19 104.7246 0)
+			(at 123.19 102.1846 0)
 			(effects
 				(font
@@
 		)
 		(pin "CHA" input
-			(at 149.86 96.52 0)
+			(at 149.86 93.98 0)
 			(effects
 				(font
@@
 		)
 		(pin "CHB" input
-			(at 149.86 99.06 0)
+			(at 149.86 96.52 0)
 			(effects
 				(font
@@
 		)
 		(pin "SW" input
-			(at 149.86 101.6 0)
+			(at 149.86 99.06 0)
 			(effects
 				(font
