File: Touchpoint_Mainboard/Touchpoint_Mainboard.kicad_pcb (KiCad board)
At the start: 2 copper layers, 58 x 96.4 mm, 99 parts, among them J101 Conn_01x02, J201 USB4105-GF-A, J602 Conn_01x11, J701 Conn_01x32, J702 Conn_01x32, SW801 SW_SPST, SW802 SW_SPST, SW803 SW_SPST, U101 RP2040, U102 NCP1117-3.3_SOT223, U103 W25Q128JVS, U201 USBLC6-2SC6, U301 Val**, U302 TLS105B0MBHTSA1, U401 DRV2605LDGS, U501 BNO055, U701 HV507PG-G, Y101 ABM8-272-T3, Y501 Crystal

Commit message: Final changes for manufacturing
Parts:
- moved C103 0.28 mm to (65.7, 37.5)
- moved C104 0.28 mm to (66.9, 37.5)
Routing:
- net /GPIO23: track 62.8 -> 65.0 mm
- net +1V1: track 22.6 -> 21.2 mm
- net /GPIO17: track 72.2 -> 73.4 mm
- net GND: track 83.5 -> 84.6 mm
- net /GPIO26: track 103.3 -> 104.1 mm
- net /GPIO29: track 82.6 -> 83.2 mm
- net /BNO085/PS1: track 6.18 -> 6.75 mm
- net /GPIO27: track 98.3 -> 98.8 mm
- net /GPIO16: track 77.3 -> 77.8 mm

Commit message: Final manufacturing adjustments
Parts:
- added C804: 0.1u, Capacitor_SMD:C_0402_1005Metric, F.Cu at (58.0, 90.1)
- added C805: 0.1u, Capacitor_SMD:C_0402_1005Metric, F.Cu at (71.0, 95.8)
- added C806: 0.1u, Capacitor_SMD:C_0402_1005Metric, F.Cu at (67.0, 98.5)
- added R804: 10k, Resistor_SMD:R_0402_1005Metric, F.Cu at (58.0, 88.9)
- added R805: 10k, Resistor_SMD:R_0402_1005Metric, F.Cu at (69.8, 95.8)
- added R806: 10k, Resistor_SMD:R_0402_1005Metric, F.Cu at (68.2, 98.5)
- C103, C105: footprint Capacitor_SMD:C_0402_1005Metric -> Capacitor_SMD:C_0805_2012Metric
- J602: value Conn_01x11 -> Conn_01x10; footprint Touchpoint:Jumper_Interface_11 -> Touchpoint:Jumper_Interface_10
- U301: value Val** -> PMW3360DM
- moved J602 2.50 mm to (42.9, 113.6)
- moved C103 2.02 mm to (63.7, 37.8)
- moved C105 1.71 mm to (60.3, 39.7)
- moved G*** 1.51 mm to (51.2, 95.8)
Connections:
- J602 pad 10: /GPIO17 -> /GPIO18
- J602 pad 2: +3.3V -> VBUS
- J602 pad 3: VBUS -> VPP
- J602 pad 4: VPP -> /GPIO28
- J602 pad 5: /GPIO28 -> /GPIO29
- J602 pad 6: /GPIO29 -> /GPIO14
- J602 pad 7: /GPIO14 -> /GPIO8
- J602 pad 8: /GPIO8 -> /GPIO16
- J602 pad 9: /GPIO16 -> /GPIO17
Routing:
- net +3.3V: track 333.8 -> 344.3 mm
- net +1V1: track 21.2 -> 26.1 mm, vias 2 -> 4
- net GND: track 84.6 -> 87.8 mm, vias 104 -> 109
- net /QSPI_SS: track 20.3 -> 17.4 mm
- net /GPIO17: track 73.4 -> 76.2 mm, vias 1 -> 2
- net /GPIO18: track 73.2 -> 75.7 mm, vias 1 -> 2
- net /QSPI_SD0: track 10.8 -> 8.99 mm
- net /QSPI_SCLK: track 13.9 -> 12.0 mm
- net /QSPI_SD3: track 15.3 -> 13.6 mm
- net /QSPI_SD1: track 11.7 -> 12.2 mm
- net /GPIO10: track 45.3 -> 45.8 mm
Other:
- board text added: "CHRG"
- board text added: "GND"
- board text added: "NEOPIX"
- board text added: "RCLCK"
- board text added: "SCRLA"
- board text added: "SCRLB"
- board text added: "SERVO"
- board text added: "VBUS"
- board text added: "VPP"
- board text added: "VREF"

Commit message: Fixed EEOP via size
Parts:
- U301: value PMW3360DM -> Val**
Changed lines of the file:
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@@
 	(generator_version "9.0")
 	(general
-		(thickness 1.6)
+		(thickness 1.67)
 		(legacy_teardrops no)
 	)
@@
 	)
 	(setup
+		(stackup
+			(layer "F.SilkS"
+				(type "Top Silk Screen")
+			)
+			(layer "F.Paste"
+				(type "Top Solder Paste")
+			)
+			(layer "F.Mask"
+				(type "Top Solder Mask")
+				(thickness 0.01)
+			)
+			(layer "F.Cu"
+				(type "copper")
+				(thickness 0.035)
+			)
+			(layer "dielectric 1"
+				(type "core")
+				(thickness 1.58)
+				(material "FR4")
+				(epsilon_r 4.5)
+				(loss_tangent 0.02)
+			)
+			(layer "B.Cu"
+				(type "copper")
+				(thickness 0.035)
+			)
+			(layer "B.Mask"
+				(type "Bottom Solder Mask")
+				(thickness 0.01)
+			)
+			(layer "B.Paste"
+				(type "Bottom Solder Paste")
+			)
+			(layer "B.SilkS"
+				(type "Bottom Silk Screen")
+			)
+			(copper_finish "None")
+			(dielectric_constraints no)
+		)
 		(pad_to_mask_clearance 0)
 		(allow_soldermask_bridges_in_footprints no)
@@
 			)
 		)
-		(property "Value" "PMW3360DM"
+		(property "Value" "Val**"
 			(at 0 0 90)
 			(layer "F.Fab")
@@
 		(model "C:/Users/carso/Documents/GitHub/Touchpoint-Mouse/Touchpoint-PCB/models/PMW3360 v12 v1.step"
 			(offset
-				(xyz -5.675 -5.35 3)
+				(xyz -5.675 -5.35 2.125)
 			)
 			(scale
