File: Touchpoint_Topboard/Touchpoint_Topboard.kicad_sch (KiCad schematic)
At the start: 13 parts, among them J1 Conn_01x03, J2 Conn_01x03, J4 EC10E1220501, J5 Conn_01x11, SW3 SW_SPST, U101 AS78L05RTR-E1

Commit message: Finished adjusting mechanical components
Connections:
- net GND: now also J4.1; no longer J4.2
- net SCROLLA: now also J4.3; no longer J4.1
- net SCROLLB: now also J4.2; no longer J4.3
Changed lines of the file:
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@@
 	)
 	(label "SCROLLA"
-		(at 90.17 55.88 180)
+		(at 90.17 60.96 180)
 		(effects
 			(font
@@
 	)
 	(label "SCROLLB"
-		(at 90.17 60.96 180)
+		(at 90.17 58.42 180)
 		(effects
 			(font
@@
 	(symbol
 		(lib_id "power:GND")
-		(at 90.17 58.42 270)
+		(at 90.17 55.88 270)
 		(unit 1)
 		(exclude_from_sim no)
@@
 		(fields_autoplaced yes)
 		(property "Reference" "#PWR011"
-			(at 83.82 58.42 0)
+			(at 83.82 55.88 0)
 			(effects
 				(font
@@
 		)
 		(property "Value" "GND"
-			(at 86.36 58.4199 90)
+			(at 86.36 55.8799 90)
 			(effects
 				(font
@@
 		)
 		(property "Footprint" ""
-			(at 90.17 58.42 0)
+			(at 90.17 55.88 0)
 			(effects
 				(font
@@
 		)
 		(property "Datasheet" ""
-			(at 90.17 58.42 0)
+			(at 90.17 55.88 0)
 			(effects
 				(font
@@
 		)
 		(property "Description" "Power symbol creates a global label with name \"GND\" , ground"
-			(at 90.17 58.42 0)
+			(at 90.17 55.88 0)
 			(effects
 				(font

Commit message: Final manufacturing adjustments
Parts:
- removed C35: 0.1u, Capacitor_SMD:C_0402_1005Metric, symbol Device:C_Small
- removed J5: Conn_01x11, Touchpoint:Jumper_Interface_11, symbol Connector_Generic:Conn_01x11
- removed R24: 10k, Resistor_SMD:R_0402_1005Metric, symbol Device:R
- added J101: Conn_01x10, Touchpoint:Jumper_Interface_10, symbol Connector_Generic:Conn_01x10
Connections:
- net +5V: now also D2.2 (A)
- net CHARGE: now also J101.5 (Pin_5)
- net GND: now also J101.1 (Pin_1)
- net NEOPIXEL: now also J101.7 (Pin_7)
- net RCLICK: now also J101.8 (Pin_8)
- net SCROLLA: now also J101.9 (Pin_9)
- net SCROLLB: now also J101.10 (Pin_10)
- net SERVO: now also J101.6 (Pin_6)
- net VBUS: now also J101.2 (Pin_2); no longer D2.2 (A)
- net VPP: now also J101.3 (Pin_3)
- net VREF: now also J101.4 (Pin_4)
Other:
- moved on the sheet: SW3
