File: Touchpoint_Topboard/Touchpoint_Topboard.kicad_pcb (KiCad board)
At the start: 2 copper layers, 51 x 96.4 mm, 35 parts, among them J1 Conn_01x03, J2 Conn_01x03, J4 EC10E1220501, J5 Conn_01x11, Q1 NMOS, SW3 SW_SPST, U1 LT3750AEMS-TRPBF, U101 AS78L05RTR-E1, U201 DA2032-AL

Commit message: Finished adjusting mechanical components
Parts:
- moved J4 10.8 mm to (60.1, 34.5), turned to 90 degrees
- moved SW3 1.47 mm to (68.0, 33.6), turned to 90 degrees
- moved R24 0.92 mm to (71.7, 39.5)
- moved C35 0.92 mm to (70.2, 39.5)
Connections:
- J4 pad 1: /SCROLLA -> GND
- J4 pad 2: GND -> /SCROLLB
- J4 pad 3: /SCROLLB -> /SCROLLA
Routing:
- net /RCLICK: track 101.0 -> 90.8 mm
- net /SCROLLB: track 89.7 -> 84.5 mm
- net GND: track 66.4 -> 63.4 mm, vias 41 -> 33
- net /SCROLLA: track 92.3 -> 89.6 mm
- net +3.3V: track 88.7 -> 87.5 mm
Other:
- board size 51 x 96.4 mm -> 51 x 96 mm

Commit message: Final changes for manufacturing
Routing:
- net /SCROLLB: track 84.5 -> 86.7 mm
- net /SCROLLA: track 89.6 -> 90.2 mm
Changed lines of the file:
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@@
 			(outputformat 1)
 			(mirror no)
-			(drillshape 1)
+			(drillshape 0)
 			(scaleselection 1)
-			(outputdirectory "")
+			(outputdirectory "./fab")
 		)
 	)
@@
 		)
 		(group ""
-			(members "01420125-4066-44da-939c-ec5ff5b74ad0" "153e1809-f56b-4380-8fbf-549e41e90e4a"
-				"1f629c5c-bbe8-4199-953f-2ce67ebfe381" "1fa868d0-7630-465a-a023-9f2011d34163"
-				"367838ff-b4cc-4f92-9241-615470c16196" "39827102-e741-4fae-9810-b72806159da4"
-				"3e1e6375-33c6-4d84-8e44-c0b0839358d9" "4dd426a6-3588-411a-95a6-5fd66209c2e8"
-				"609a32ba-b8c8-40ee-9f5f-8a0d88addf8d" "686980c9-dd61-477f-a935-0cf9d4d12622"
-				"69ab94a6-b8d6-4cd6-ab44-95c923633278" "7247e2ab-7433-49a7-a75f-d081b18df009"
-				"7ab925c5-c6d0-4cd5-974a-622107fcd906" "83a06213-25cb-405b-b37f-e9d18e881dd9"
-				"8a7b7f93-5791-4b94-8a92-df2aaffa4242" "9bdb273f-77db-4c0d-98d0-0a0281aacc3c"
-				"ae65fdb6-f524-468e-8716-f5d58c166b24" "b6cf7828-ac1e-4cd5-b433-50e5c162e8b2"
-				"c20183c7-203a-4723-a0e6-d3e097821bc4" "d4f2c94c-7df2-4794-83db-fe139eb92271"
-				"d598dc3b-7afe-48ba-aeda-92a6805c1757" "d87c5930-e517-4fee-98e1-886e87d0b18c"
-				"f4c5831b-0d91-4835-ab94-383df5a5b851" "ffff58e3-ceab-4484-ad5f-9c96f45e628f"
+			(members "09fc1074-3dc3-4a29-9581-1db7ab30f307" "1911a467-39a8-45f8-ac0b-ffa15facbe87"
+				"34394bdd-e48f-4787-8a2f-4a3f07fc0192" "37c1b46f-b8f9-49a1-9aeb-c046f797b89d"
+				"5036b3d5-f6b4-47cf-92d4-2c2b7b25de50" "52c0e6e4-9077-4abc-997b-2076fabcbf30"
+				"5e978fc1-9797-4410-a2f5-e346719d1e8a" "6b9c75d3-d675-4dae-87e4-9845e490c132"
+				"6d7dfb6c-5e4d-4b61-9f09-85384c4261e8" "71986d23-e4c9-4f0e-b55d-a268ecfebe28"
+				"7a612717-32f2-4890-a8a5-ccc12393973a" "88bcdaa8-b348-4b63-a73b-b7dec04da65d"
+				"90ec6b15-0d71-4b30-afe8-d42a86676607" "a3940e08-4fe5-435c-804f-54a6ed53c937"
+				"a3e900e9-a241-4a49-88cf-df5706a3b25a" "a7118d91-3a8f-48d8-b5c2-19a748fba31f"
+				"b2edca90-e9f0-499d-8004-391ff7079d4e" "beb7475f-2363-48d8-9853-d61a1696205a"
+				"c6789c08-2377-4f67-a030-92a983437a82" "c6d26c39-13f0-49a1-983b-0d5909e45d4f"
+				"c7754f9a-a888-47a5-9ea8-c8fbe1b37091" "e4e37896-3b3d-4716-9743-25f35149d431"
+				"f3208f61-30ed-4b07-8336-f92c4307cb17" "fda58136-0f94-4f4a-b2cd-9c0366b72ff4"
 			)
 		)
@@
 			(net 1 "GND")
 			(pintype "passive")
-			(solder_mask_margin 0.102)
+			(solder_mask_margin 0)
 		)
 		(pad "P$2" smd rect
@@
 			(size 3.43 1.79)
 			(layers "F.Cu" "F.Mask" "F.Paste")
-			(solder_mask_margin 0.102)
+			(solder_mask_margin 0)
 		)
 		(pad "P$3" smd rect
@@
 			(net 24 "unconnected-(U201-PadP$3)")
 			(pintype "passive+no_connect")
-			(solder_mask_margin 0.102)
+			(solder_mask_margin 0)
 		)
 		(pad "P$4" smd rect
@@
 			(net 27 "unconnected-(U201-PadP$4)")
 			(pintype "passive+no_connect")
-			(solder_mask_margin 0.102)
+			(solder_mask_margin 0)
 		)
 		(pad "P$5" smd rect
@@
 			(net 16 "Net-(Q1-D)")
 			(pintype "passive")
-			(solder_mask_margin 0.102)
+			(solder_mask_margin 0)
 		)
 		(pad "P$6" smd rect
@@
 			(net 16 "Net-(Q1-D)")
 			(pintype "passive")
-			(solder_mask_margin 0.102)
+			(solder_mask_margin 0)
 		)
 		(pad "P$7" smd rect
@@
 			(net 2 "+5V")
 			(pintype "passive")
-			(solder_mask_margin 0.102)
+			(solder_mask_margin 0)
 		)
 		(pad "P$8" smd rect
@@
 			(net 2 "+5V")
 			(pintype "passive")
-			(solder_mask_margin 0.102)
+			(solder_mask_margin 0)
 		)
 		(pad "P$9" smd rect
@@
 			(net 26 "unconnected-(U201-PadP$9)")
 			(pintype "passive+no_connect")
-			(solder_mask_margin 0.102)
+			(solder_mask_margin 0)
 		)
 		(pad "P$10" smd rect
@@
 			(net 25 "unconnected-(U201-PadP$10)")
 			(pintype "passive+no_connect")
-			(solder_mask_margin 0.102)
+			(solder_mask_margin 0)
 		)
 		(pad "P$11" smd rect
@@
 			(size 3.43 1.79)
 			(layers "F.Cu" "F.Mask" "F.Paste")
-			(solder_mask_margin 0.102)
+			(solder_mask_margin 0)
 		)
 		(pad "P$12" smd rect
@@
 			(net 6 "Net-(D1-A)")
 			(pintype "passive")
-			(solder_mask_margin 0.102)
+			(solder_mask_margin 0)
 		)
 		(embedded_fonts no)
@@
 			(pintype "unspecified")
 		)
-		(pad "4" smd rect
+		(pad "4" thru_hole oval
 			(at -1.999999 2.000001 90)
-			(size 1.8034 2.0066)
-			(layers "F.Cu" "F.Mask" "F.Paste")
+			(size 2.3 2.7)
+			(drill oval 1.8 2.2)
+			(layers "*.Cu" "*.Mask")
+			(remove_unused_layers no)
 		)
-		(pad "5" smd rect
+		(pad "5" thru_hole oval
 			(at 6.999999 2.000001 90)
-			(size 1.8034 2.0066)
-			(layers "F.Cu" "F.Mask" "F.Paste")
+			(size 2.3 2.7)
+			(drill oval 1.8 2.2)
+			(layers "*.Cu" "*.Mask")
+			(remove_unused_layers no)
 		)
 		(embedded_fonts no)
@@
 	)
 	(segment
-		(start 57.74962 85.49962)
-		(end 65.751 93.501)
+		(start 65.751 93.501)
+		(end 65.751 109.849)
 		(width 0.2)
 		(layer "B.Cu")
@@
 	)
 	(segment
-		(start 65.751 109.849)
-		(end 64.6 111)
+		(start 57 32.61)
+		(end 57 84.75)
 		(width 0.2)
 		(layer "B.Cu")
@@
 	)
 	(segment
-		(start 57.74962 31.86038)
-		(end 57.74962 85.49962)
+		(start 57 84.75)
+		(end 65.751 93.501)
 		(width 0.2)
 		(layer "B.Cu")
@@
 	)
 	(segment
-		(start 65.751 93.501)
-		(end 65.751 109.849)
+		(start 65.751 109.849)
+		(end 64.6 111)
 		(width 0.2)
 		(layer "B.Cu")
@@
 	(segment
 		(start 60.11 29.5)
-		(end 57.74962 31.86038)
+		(end 57 32.61)
 		(width 0.2)
 		(layer "B.Cu")
@@
 	)
 	(segment
-		(start 62.5 89.5)
-		(end 62.5 34.39)
+		(start 66 111.6)
+		(end 66.25 111.35)
 		(width 0.2)
 		(layer "B.Cu")
@@
 	)
 	(segment
-		(start 66 111.6)
-		(end 66.25 111.35)
+		(start 66.25 111.35)
+		(end 66.25 93.25)
 		(width 0.2)
 		(layer "B.Cu")
@@
 	)
 	(segment
-		(start 66.25 93.25)
-		(end 62.5 89.5)
+		(start 57.5 34.61)
+		(end 60.11 32)
 		(width 0.2)
 		(layer "B.Cu")
@@
 	)
 	(segment
-		(start 62.5 34.39)
-		(end 60.11 32)
+		(start 57.5 84.5)
+		(end 57.5 34.61)
 		(width 0.2)
 		(layer "B.Cu")
@@
 	)
 	(segment
-		(start 66.25 111.35)
-		(end 66.25 93.25)
+		(start 66.25 93.25)
+		(end 57.5 84.5)
 		(width 0.2)
 		(layer "B.Cu")

Commit message: Final manufacturing adjustments
Parts:
- removed C35: 0.1u, Capacitor_SMD:C_0402_1005Metric
- removed J5: Conn_01x11, Touchpoint:Jumper_Interface_11
- removed R24: 10k, Resistor_SMD:R_0402_1005Metric
- added J101: Conn_01x10, Touchpoint:Jumper_Interface_10, F.Cu at (42.9, 113.6)
- moved D2 15.2 mm to (46.2, 99.5)
- moved D3 12.9 mm to (46.2, 102.2)
- moved R7 12.7 mm to (49.0, 99.5), turned to 0 degrees
- moved R10 10.9 mm to (49.0, 102.2)
Connections:
- D2 pad 2: VBUS -> +5V
Routing:
- net +3.3V: track 87.5 -> 0.00 mm, vias 2 -> 0
- net VBUS: track 60.8 -> 42.9 mm
- net /CHARGE: track 28.6 -> 41.7 mm, vias 0 -> 2
- net GND: track 63.4 -> 57.7 mm, vias 33 -> 31
- net +5V: track 52.7 -> 58.3 mm
Other:
- outline, holes or cut-outs redrawn
- board text added: "CHRG"
- board text added: "NEOPIX"
- board text added: "RCLCK"
- board text added: "SCRLA"
- board text added: "SCRLB"
- board text added: "SERVO"
- board text added: "VPP"
- board text added: "VREF"
- board text removed: "CHARGE"
